File: SpinnerLights/Board/SpinnerLights.sch (KiCad schematic (older format))
At the start: 14 parts, among them U1 SeeeduinoXIAO, U2 ADXL343

Commit message: SpinnerLights: Fix symbols for NeoPixels
Parts:
- PIXEL2, PIXEL3, PIXEL4, Pixel1: value NeoPixel_THT -> SK6812MINI; symbol LED:NeoPixel_THT -> LED:SK6812MINI
Changed lines of the file:
@@
 	5450 4250 5300 4250
 $Comp
-L LED:NeoPixel_THT Pixel1
+L LED:SK6812MINI Pixel1
 U 1 1 6169F8F8
 P 8900 1600
 F 0 "Pixel1" V 8854 1944 50  0000 L CNN
-F 1 "NeoPixel_THT" V 8945 1944 50  0000 L CNN
+F 1 "SK6812MINI" V 8945 1944 50  0000 L CNN
 F 2 "LED_SMD:LED_SK6812MINI_PLCC4_3.5x3.5mm_P1.75mm" H 8950 1300 50  0001 L TNN
 F 3 "https://www.adafruit.com/product/1938" H 9000 1225 50  0001 L TNN
@@
 $EndComp
 $Comp
-L LED:NeoPixel_THT PIXEL4
+L LED:SK6812MINI PIXEL4
 U 1 1 616C9B9C
 P 10350 1600
 F 0 "PIXEL4" V 10396 1256 50  0000 R CNN
-F 1 "NeoPixel_THT" V 10305 1256 50  0000 R CNN
+F 1 "SK6812MINI" V 10305 1256 50  0000 R CNN
 F 2 "LED_SMD:LED_SK6812MINI_PLCC4_3.5x3.5mm_P1.75mm" H 10400 1300 50  0001 L TNN
 F 3 "https://www.adafruit.com/product/1938" H 10450 1225 50  0001 L TNN
@@
 	8600 2700 8600 1600
 Connection ~ 8600 2700
-$Comp
-L LED:NeoPixel_THT PIXEL2
-U 1 1 616B291A
-P 8900 2700
-F 0 "PIXEL2" V 8854 3044 50  0000 L CNN
-F 1 "NeoPixel_THT" V 8945 3044 50  0000 L CNN
-F 2 "LED_SMD:LED_SK6812MINI_PLCC4_3.5x3.5mm_P1.75mm" H 8950 2400 50  0001 L TNN
-F 3 "https://www.adafruit.com/product/1938" H 9000 2325 50  0001 L TNN
-	1    8900 2700
-	0    1    1    0
-$EndComp
 Wire Wire Line
 	8600 2700 8600 3050
@@
 Connection ~ 10650 2700
 $Comp
-L LED:NeoPixel_THT PIXEL3
+L LED:SK6812MINI PIXEL3
 U 1 1 6175018F
 P 10350 2700
 F 0 "PIXEL3" V 10396 2356 50  0000 R CNN
-F 1 "NeoPixel_THT" V 10305 2356 50  0000 R CNN
+F 1 "SK6812MINI" V 10305 2356 50  0000 R CNN
 F 2 "LED_SMD:LED_SK6812MINI_PLCC4_3.5x3.5mm_P1.75mm" H 10400 2400 50  0001 L TNN
 F 3 "https://www.adafruit.com/product/1938" H 10450 2325 50  0001 L TNN
@@
 Text Label 8200 4350 0    50   ~ 0
 B15
+$Comp
+L LED:SK6812MINI PIXEL2
+U 1 1 616B291A
+P 8900 2700
+F 0 "PIXEL2" V 8854 3044 50  0000 L CNN
+F 1 "SK6812MINI" V 8945 3044 50  0000 L CNN
+F 2 "LED_SMD:LED_SK6812MINI_PLCC4_3.5x3.5mm_P1.75mm" H 8950 2400 50  0001 L TNN
+F 3 "https://www.adafruit.com/product/1938" H 9000 2325 50  0001 L TNN
+	1    8900 2700
+	0    1    1    0
+$EndComp
 $EndSCHEMATC
